File: Robot/Électronique/image/doom_v1.kicad_sch (KiCad schematic)
At the start: 265 parts, among them J1 STEPPER G, J10 Conn_01x04, J11 Conn_01x04, J12 Conn_01x04, J13 Conn_01x04, J14 Conn_01x04, J15 Conn_01x04, J16 Conn_01x04, J17 Conn_01x04, J18 Conn_01x04, J19 Conn_01x04, J2 STEPPER 1, J20 Conn_01x04, J21 Conn_01x04, J22 Conn_01x04, J23 Conn_01x02, J24 Conn_01x02, J25 Conn_01x02, J26 Conn_01x02, J27 Conn_01x02, J28 Conn_01x02, J29 Conn_01x02, J3 STEPPER 3, J30 Conn_01x02, J31 Conn_02x04_Odd_Even, J32 Conn_02x04_Odd_Even, J33 Conn_02x04_Odd_Even, J34 Conn_02x04_Odd_Even, J35 Conn_02x04_Odd_Even, J36 Conn_02x04_Odd_Even, J37 Conn_02x04_Odd_Even, J38 Conn_02x04_Odd_Even, J39 Conn_02x04_Odd_Even, J4 STEPPER D, J40 Conn_02x04_Odd_Even, J41 Conn_02x04_Odd_Even, J42 Conn_02x04_Odd_Even, J43 I2C Extension, J44 I2C Extension, J45 UART BONUS, J46 con AX12A, J47 gyro, J48 ventilo 1, J49 ventilo 2, J5 STEPPER 2, J50 LIDAR, J51 XBEE, J6 STEPPER 4, J7 Conn_01x04, J8 Conn_01x04, J9 Conn_01x04, K1 TE_PCH-1xxx2M, U1 TMC2209_SILENTSTEPSTICK, U10 XIAO-HALF-HOLE-23P, U11 PCF8574AT, U12 PCF8574AT, U13 PCF8574AT, U14 TFT_320x240, U15 XIAO-HALF-HOLE-23P, U16 TSR1-2433E, U17 TSR1-2450E, U18 TSR1-2450E, U19 XIAO-ESP32-S3-DIP, U2 TMC2209_SILENTSTEPSTICK, U3 TMC2209_SILENTSTEPSTICK, U4 TMC2209_SILENTSTEPSTICK, U5 TMC2209_SILENTSTEPSTICK, U6 TMC2209_SILENTSTEPSTICK, U7 PCA9685PW, U8 PCA9685PW, U9 PCA9685PW

Commit message: avancement
Other:
- note added: "Connecteurs"
- note added: "Convertisseur puissance actionneur"
- note added: "Convertisseur puissance logique"
- note added: "Driver pour moteurs Pas à Pas"
- note added: "Extension analogique"
- note added: "Extension pour Boutons/Switch"
- note added: "LED d'états"
- note added: "LED témoins"
- note added: "Micro controlleurs"
- note added: "Module extension Servo/Pompe"
- note added: "Trou de montage"
- note added: "connecteur alimentation"
- note added: "connecteur extensions"
- note added: "relais externe"
- note added: "ventilo"
- note added: "Écran tactile"
- company: (none) -> Unimakers
- title: (none) -> Schéma doom
- moved on the sheet: BZ1, Batcon1, Batcon2, Bau.1, C1, C10, C11, C13, C15, C2, C3, C4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
